Commit message: Gazebo Simulation V1.0.0

File: description/robot.urdf.xacro (robot description, xacro)
@@ -4,3 +4,5 @@
     <xacro:include filename="$(find gazebo_bot_sim-)/description/robot_core.xacro"/>
     <!-- <link name="base_link"></link> -->
+    <xacro:include filename="$(find gazebo_bot_sim-)/description/gazebo_control.xacro"/>
+    <xacro:include filename="$(find gazebo_bot_sim-)/description/lidar.xacro"/>
 </robot>

File: description/robot_core.xacro (robot description, xacro)
@@ -14,6 +14,17 @@
         <color rgba="0 0 0 1"/>
     </material>
+    <material name="red">
+        <color rgba="1 0 0 1"/>
+    </material>
     <!-- BASE LINK -->
     <link name="base_link">
+    </link>
+    <!-- BASE FOOTPRINT LINK -->
+    <joint name="base_footprint_joint" type="fixed">
+        <parent link="base_link"/>
+        <child link="base_footprint"/>
+        <origin xyz="0 0 0" rpy="0 0 0"/>
+    </joint>
+    <link name="base_footprint">
     </link>
     <!-- CHASSIS LINK -->
@@ -42,4 +53,7 @@
         </xacro:inertial_box>
     </link>
+    <gazebo referrence="chassis">
+        <material>Gazebo/White</material>
+    </gazebo>
     <!-- LEFT WHEEL LINK  -->
     <joint name="left_wheel_joint" type="continuous">
@@ -66,4 +80,7 @@
         </xacro:inertial_cylinder>
     </link>
+    <gazebo referrence="left_wheel">
+        <material>Gazebo/Blue</material>
+    </gazebo>
     <!-- RIGHT WHEEL LINK  -->
     <joint name="right_wheel_joint" type="continuous">
@@ -90,4 +107,7 @@
         </xacro:inertial_cylinder>
     </link>
+    <gazebo referrence="right_wheel">
+        <material>Gazebo/Blue</material>
+    </gazebo>
     <!-- CASTER WHEEL LINK  -->
     <joint name="caster_wheel_joint" type="fixed">
@@ -113,3 +133,8 @@
         </xacro:inertial_sphere>
     </link>
+    <gazebo reference="caster_wheel">
+        <material>Gazebo/White</material>
+        <mu1 value="0.001"/>
+        <mu2 value="0.001"/>
+    </gazebo>
 </robot>
